Commit message: added camera (visualization)

File: robutler_description/urdf/robutler.gazebo.xacro (robot description, xacro)
@@ -6,4 +6,7 @@
   <gazebo reference="base_link">
     <material>Gazebo/DarkGrey</material>
+  </gazebo>
+  <gazebo reference ="camera_link">
+      <material>Gazebo/DarkGrey</material>
   </gazebo>
   <gazebo reference="wheel_left_link">
@@ -137,5 +140,5 @@
   </gazebo>
   <!-- my second lidar -->
-  <gazebo reference="base_2_scan">
+  <!-- <gazebo reference="base_2_scan">
     <material>Gazebo/FlatBlack</material>
     <sensor type="ray" name="lds_lfcd_sensor">
@@ -168,5 +171,5 @@
       </plugin>
     </sensor>
-  </gazebo>
+  </gazebo> -->
 <!--link : https://www.raspberrypi.org/documentation/hardware/camera/-->
   <gazebo reference="camera_rgb_frame">

File: robutler_description/urdf/robutler.urdf.xacro (robot description, xacro)
@@ -161,32 +161,4 @@
   </link>
   <!-- TODO insert new lidar in an higher position-->
-  <joint name="scan_2_joint" type="fixed">
-    <parent link="base_link"/>
-    <child link="base_2_scan"/>
-    <!-- <origin xyz="-0.064 0 0.122" rpy="0 0 0"/> -->
-    <origin xyz="-0.064 0 0.222" rpy="0 0 0"/>
-  </joint>
-  <link name="base_2_scan">
-    <visual>
-      <origin xyz="0 0 0.0" rpy="0 0 0"/>
-      <geometry>
-        <mesh filename="package://turtlebot3_description/meshes/sensors/lds.stl" scale="0.001 0.001 0.001"/>
-      </geometry>
-      <material name="dark"/>
-    </visual>
-    <collision>
-      <origin xyz="0.015 0 -0.0065" rpy="0 0 0"/>
-      <geometry>
-        <cylinder length="0.0315" radius="0.055"/>
-      </geometry>
-    </collision>
-    <inertial>
-      <mass value="0.114" />
-      <origin xyz="0 0 0" />
-      <inertia ixx="0.001" ixy="0.0" ixz="0.0"
-               iyy="0.001" iyz="0.0"
-               izz="0.001" />
-    </inertial>
-  </link>
   <joint name="camera_joint" type="fixed">
     <!-- <origin xyz="0.073 -0.011 0.084" rpy="0 0 0"/> -->
@@ -201,4 +173,11 @@
       <geometry>
         <cylinder length="0.584" radius="0.01"/>
+      </geometry>
+      <material name="dark"/>
+    </visual>
+    <visual>
+      <origin xyz="0.03 0.011 0.01" rpy="0 0 0"/>
+      <geometry>
+        <box size="0.1 0.05 0.05" />
       </geometry>
       <material name="dark"/>
